Commit message: Added an extra x1_gazebo xacro file and fixed problem of wheel rotating on its own

File: src/x1_description/urdf/x1.urdf.xacro (robot description, xacro)
@@ -1,4 +1,6 @@
 <?xml version = "1.0"?>
-<robot xmlns:xacro="http://www.ros.org/wiki/xacro" name = "ROSMASTER_X1">
+<robot name = "ROSMASTER_X1" xmlns:xacro="http://www.ros.org/wiki/xacro">
+    <!-- Include Gazebo Parameters -->
+    <xacro:include filename="$(find x1_description)/urdf/x1_gazebo.xacro" />
     <!-- Material definitions -->
     <material name="Green">
@@ -37,4 +39,5 @@
             <axis xyz="${axis}"/>
             <limit lower="${-pi}" upper="${pi}" effort="100" velocity="1"/>
+            <dynamics friction="1E-04"/>
         </joint>
     </xacro:macro>
@@ -62,5 +65,5 @@
     </xacro:common_link>
     <!-- Fixed Joints -->
-    <xacro:fixed_joint name="base_joint" parent="base_footprint" child="base_link" xyz="0.0 0.0 0.0815" rpy="0 0 0"/>
+    <xacro:fixed_joint name="base_joint" parent="base_footprint" child="base_link" xyz="0.0 0.0 0.0850" rpy="0 0 0"/>
     <link name="imu_link"/>
     <xacro:fixed_joint name="base_imu" parent="base_link" child="imu_link" xyz="-0.06 0.01 0.01" rpy="0 3.1415 1.5707"/>

Commit message: robot moves in response to joystick command in Gazebo simulation and RViz
Simulation work on the computer to get the Gazebo and RViz robot simulation to move using a DiffDriveController.
- added a dummy JointGroupVelocityController named simple_velocity_controller in controller_manager to investigate the reason behind DiffDriveController not working. When using the simple_velocity_controller and publishing Float64MultiArray onto the /simple_velocity_controller/commands topic, the robot moves. It turns out that I must send TwistStamped messages (with time stampe and frame in the header) to /x1_controller/cmd_vel for the simulation to work
- display.launch.py now only brings up RViz since the joint_state_broadcaster controller controller already broadcast the joint states. When they were launched along with RViz, there were missing transforms between the odom frame and the wheels because these nodes were overriding the joint_state_broadcaster controller.
- fixed the axis of rotation in the URDF file for the left wheels (This led to a problem where the Gazebo and RViz simulation would have completely different motion)
- new mesh for the base_link.stl without the screen (from Matt's repo)

Updated the dev container to automatically source the workspace when a new terminal is opened

File: src/x1_description/urdf/x1.urdf.xacro (robot description, xacro)
@@ -98,5 +98,5 @@
     </xacro:common_link>
     <xacro:continuous_joint name="front_left_joint" parent="base_link" child="front_left_wheel"
-                      xyz="0.08 0.084492 -0.0389" rpy="${pi/2} 0 0" axis="0 0 1"/>
+                      xyz="0.08 0.0845 -0.0389" rpy="${pi/2} 0 0" axis="0 0 -1"/>
     <xacro:common_link name="back_right_wheel" material="White" path="mecanum" collision_shape="cylinder" collision_size="0.035 0.03">
         <inertial>
@@ -108,5 +108,5 @@
     </xacro:common_link>
     <xacro:continuous_joint name="back_right_joint" parent="base_link" child="back_right_wheel"
-                      xyz="-0.08 -0.0845 -0.03946" rpy="-${pi/2} 0 0" axis="0 0 1"/>
+                      xyz="-0.08 -0.0845 -0.0395" rpy="-${pi/2} 0 0" axis="0 0 1"/>
     <xacro:common_link name="back_left_wheel" material="White" path="mecanum" collision_shape="cylinder" collision_size="0.035 0.03">
         <inertial>
@@ -118,5 +118,5 @@
     </xacro:common_link>
     <xacro:continuous_joint name="back_left_joint" parent="base_link" child="back_left_wheel"
-                      xyz="-0.08 0.084492 -0.03954" rpy="${pi/2} 0 0" axis="0 0 1"/>
+                      xyz="-0.08 0.0845 -0.0395" rpy="${pi/2} 0 0" axis="0 0 -1"/>
     <!-- Sensors -->
     <xacro:common_link name="laser_link" material="White" path="sensor" collision_shape="cylinder" collision_size="0.06 0.06" collision_xyz='-0.005 0 -0.02'>

File: src/x1_description/urdf/x1_gazebo.xacro (robot description, xacro)
@@ -1,7 +1,24 @@
 <?xml version = "1.0"?>
 <robot name="ROSMASTER_X1" xmlns:xacro="http://www.ros.org/wiki/xacro">
-    <!-- Wheels -->
+    <xacro:macro name="common_joint" params="name">
+        <gazebo reference="${name}">
+            <!-- <mu1>0.1</mu1>
+            <mu2>0.1</mu2> -->
+            <mu1>0.1</mu1>        <!-- High friction coeff to avoid slipage -->
+            <mu2>0.1</mu2>
+            <kp>1.0</kp>
+            <kd>1.0</kd>
+            <minDepth>0.001</minDepth>
+            <maxVel>10</maxVel>
+            <fdir1>1 0 0</fdir1>                <!-- Direction of wheel rotation -->
+        </gazebo>
+    </xacro:macro>
+    <xacro:common_joint name="front_right_wheel"/>
+    <xacro:common_joint name="front_left_wheel"/>
+    <xacro:common_joint name="back_right_wheel"/>
+    <xacro:common_joint name="back_left_wheel"/>
+    <!-- Wheels
     <gazebo reference = "front_right_wheel">
-        <mu1>100000000000000.0</mu1>        <!-- High friction coeff to avoid slipage -->
+        <mu1>100000000000000.0</mu1>
         <mu2>100000000000000.0</mu2>
         <kp>1000000000000.0</kp>
@@ -9,8 +26,8 @@
         <minDepth>0.001</minDepth>
         <maxVel>0.1</maxVel>
-        <fdir1>1 0 0</fdir1>                <!-- Direction of wheel rotation -->
+        <fdir1>1 0 0</fdir1>
     </gazebo>
     <gazebo reference = "front_left_wheel">
-        <mu1>100000000000000.0</mu1>        <!-- High friction coeff to avoid slipage -->
+        <mu1>100000000000000.0</mu1>
         <mu2>100000000000000.0</mu2>
         <kp>1000000000000.0</kp>
@@ -18,8 +35,8 @@
         <minDepth>0.001</minDepth>
         <maxVel>0.1</maxVel>
-        <fdir1>1 0 0</fdir1>                <!-- Direction of wheel rotation -->
+        <fdir1>1 0 0</fdir1>
     </gazebo>
     <gazebo reference = "back_right_wheel">
-        <mu1>100000000000000.0</mu1>        <!-- High friction coeff to avoid slipage -->
+        <mu1>100000000000000.0</mu1>
         <mu2>100000000000000.0</mu2>
         <kp>1000000000000.0</kp>
@@ -27,8 +44,8 @@
         <minDepth>0.001</minDepth>
         <maxVel>0.1</maxVel>
-        <fdir1>1 0 0</fdir1>                <!-- Direction of wheel rotation -->
+        <fdir1>1 0 0</fdir1>
     </gazebo>
     <gazebo reference = "back_left_wheel">
-        <mu1>100000000000000.0</mu1>        <!-- High friction coeff to avoid slipage -->
+        <mu1>100000000000000.0</mu1>
         <mu2>100000000000000.0</mu2>
         <kp>1000000000000.0</kp>
@@ -36,6 +53,6 @@
         <minDepth>0.001</minDepth>
         <maxVel>0.1</maxVel>
-        <fdir1>1 0 0</fdir1>                <!-- Direction of wheel rotation -->
-    </gazebo>
+        <fdir1>1 0 0</fdir1>
+    </gazebo> -->
     <!-- Gazebo control related stuff -->
     <gazebo>

File: src/x1_description/urdf/x1_ros2_control.xacro (robot description, xacro)
@@ -2,5 +2,5 @@
 <!-- This file configures the control plugins in the bumperbot_gazebo.xacro file -->
 <robot name = "ROSMASTER_X1" xmlns:xacro="http://www.ros.org/wiki/xacro">
-    <!-- Hardware interface for controller manager-->
+    <!-- Hardware interface for controller manager -->
     <ros2_control name = "RobotSystem" type = "system">
         <!-- If ROS2 Humble then use this plugin-->
@@ -13,5 +13,5 @@
         <xacro:unless value = "$(arg is_ignition)">
             <hardware>
-                <plugin>gz_ros2_control/GazeboSystem</plugin>
+                <plugin>gz_ros2_control/GazeboSimSystem</plugin>
             </hardware>
         </xacro:unless>

Commit message: move lidar link and joint from main URDF xacro to stand-alone xacro

File: src/x1_description/urdf/x1.urdf.xacro (robot description, xacro)
@@ -120,13 +120,5 @@
                       xyz="-0.08 0.0845 -0.0395" rpy="${pi/2} 0 0" axis="0 0 -1"/>
     <!-- Sensors -->
-    <xacro:common_link name="laser_link" material="White" path="sensor" collision_shape="cylinder" collision_size="0.06 0.06" collision_xyz='-0.005 0 -0.02'>
-        <inertial>
-            <origin xyz="-0.0176558922685589 0.000671805271544437 0.0219302095894866" rpy="0 0 0"/>
-            <mass value="0.0483909504209895"/>
-            <inertia ixx="1.58456966399128E-05" ixy="-4.23913983850005E-07" ixz="-2.09597897904374E-07"
-                     iyy="3.89262522903605E-05" iyz="3.24809725932687E-07" izz="4.86230801106223E-05"/>
-        </inertial>
-    </xacro:common_link>
-    <xacro:fixed_joint name="laser_joint" parent="base_link" child="laser_link" xyz="0.0435 5.25826986680105E-05 0.11" rpy="0 0 0"/>
+    <xacro:include filename="lidar.xacro"/>
     <xacro:common_link name="camera_link" material="White" path="sensor" collision_shape="box" collision_size="0.06 0.17 0.05">
         <inertial>

Commit message: modify camera link in URDF and add camera_optical link
- move the camera link from main URDF file to standalone file that is called in the main URDF
- add camera_optical link to match with standard image coordination frame

File: src/x1_description/urdf/x1.urdf.xacro (robot description, xacro)
@@ -121,11 +121,4 @@
     <!-- Sensors -->
     <xacro:include filename="lidar.xacro"/>
-    <xacro:common_link name="camera_link" material="White" path="sensor" collision_shape="box" collision_size="0.06 0.17 0.05">
-        <inertial>
-            <origin xyz="0 0 0" rpy="0 0 0"/>
-            <mass value="0"/>
-            <inertia ixx="0" ixy="0" ixz="0" iyy="0" iyz="0" izz="0"/>
-        </inertial>
-    </xacro:common_link>
-    <xacro:fixed_joint name="camera_joint" parent="base_link" child="camera_link" xyz="0.057105 1.7948E-05 0.03755" rpy="0 0 0"/>
+    <xacro:include filename="camera.xacro"/>
 </robot>

Commit message: change robot velocity limit for faster mapping

File: src/x1_description/urdf/x1.urdf.xacro (robot description, xacro)
@@ -48,5 +48,5 @@
             <origin xyz="${xyz}" rpy="${rpy}"/>
             <axis xyz="${axis}"/>
-            <limit lower="${-pi}" upper="${pi}" effort="100" velocity="1"/>
+            <limit lower="${-pi}" upper="${pi}" effort="100" velocity="2.5"/>
             <dynamics friction="1E-04"/>
         </joint>

File: src/x1_description/urdf/x1_gazebo.xacro (robot description, xacro)
@@ -5,6 +5,6 @@
             <!-- <mu1>0.1</mu1>
             <mu2>0.1</mu2> -->
-            <mu1>0.15</mu1>        <!-- High friction coeff to avoid slipage -->
-            <mu2>0.0</mu2>
+            <mu1>0.50</mu1>        <!-- High friction coeff to avoid slipage -->
+            <mu2>0.1</mu2>
             <kp>1.0</kp>
             <kd>1.0</kd>

File: src/x1_description/urdf/x1_ros2_control.xacro (robot description, xacro)
@@ -1,9 +1,9 @@
-<?xml version = "1.0"?>
+<?xml version="1.0"?>
 <!-- This file configures the control plugins in the bumperbot_gazebo.xacro file -->
-<robot name = "ROSMASTER_X1" xmlns:xacro="http://www.ros.org/wiki/xacro">
+<robot name="ROSMASTER_X1" xmlns:xacro="http://www.ros.org/wiki/xacro">
     <!-- Hardware interface for controller manager -->
-    <ros2_control name = "RobotSystem" type = "system">
+    <ros2_control name="RobotSystem" type="system">
         <!-- If ROS2 Humble then use this plugin-->
-        <xacro:if value = "$(arg is_ignition)">
+        <xacro:if value="$(arg is_ignition)">
             <hardware>
                 <plugin>ign_ros2_control/IgnitionSystem</plugin>
@@ -11,41 +11,55 @@
         </xacro:if>
         <!-- If higher than ROS2 Humble (Iron, Jazzy,...), then use this plugin-->
-        <xacro:unless value = "$(arg is_ignition)">
+        <xacro:unless value="$(arg is_ignition)">
             <hardware>
                 <plugin>gz_ros2_control/GazeboSimSystem</plugin>
             </hardware>
         </xacro:unless>
-        <joint name = "front_right_joint">
-            <command_interface name = "velocity">
-                <param name = "min"> -1</param>
-                <param name = "max"> 1</param>
+        <xacro:macro name="x1_control_joint" params="joint_name">
+            <joint name="${joint_name}">
+                <command_interface name="velocity">
+                    <param name="min">-5</param>
+                    <param name="max">5</param>
+                </command_interface>
+                <state_interface name="position" />
+                <state_interface name="velocity" />
+            </joint>
+        </xacro:macro>
+        <xacro:x1_control_joint joint_name="front_right_joint"></xacro:x1_control_joint>
+        <xacro:x1_control_joint joint_name="front_left_joint"></xacro:x1_control_joint>
+        <xacro:x1_control_joint joint_name="back_right_joint"></xacro:x1_control_joint>
+        <xacro:x1_control_joint joint_name="back_left_joint"></xacro:x1_control_joint>
+        <!-- <joint name="front_right_joint">
+            <command_interface name="velocity">
+                <param name="min"> -5</param>
+                <param name="max"> 5</param>
             </command_interface>
-            <state_interface name = "position"/>
-            <state_interface name = "velocity"/>
+            <state_interface name="position" />
+            <state_interface name="velocity" />
         </joint>
-        <joint name = "front_left_joint">
-            <command_interface name = "velocity">
-                <param name = "min"> -1</param>
-                <param name = "max"> 1</param>
+        <joint name="front_left_joint">
+            <command_interface name="velocity">
+                <param name="min"> -5</param>
+                <param name="max"> 5</param>
             </command_interface>
-            <state_interface name = "position"/>
-            <state_interface name = "velocity"/>
+            <state_interface name="position" />
+            <state_interface name="velocity" />
         </joint>
-        <joint name = "back_right_joint">
-            <command_interface name = "velocity">
-                <param name = "min"> -1</param>
-                <param name = "max"> 1</param>
+        <joint name="back_right_joint">
+            <command_interface name="velocity">
+                <param name="min"> -5</param>
+                <param name="max"> 5</param>
             </command_interface>
-            <state_interface name = "position"/>
-            <state_interface name = "velocity"/>
+            <state_interface name="position" />
+            <state_interface name="velocity" />
         </joint>
-        <joint name = "back_left_joint">
-            <command_interface name = "velocity">
-                <param name = "min"> -1</param>
-                <param name = "max"> 1</param>
+        <joint name="back_left_joint">
+            <command_interface name="velocity">
+                <param name="min"> -5</param>
+                <param name="max"> 5</param>
             </command_interface>
-            <state_interface name = "position"/>
-            <state_interface name = "velocity"/>
-        </joint>
+            <state_interface name="position" />
+            <state_interface name="velocity" />
+        </joint> -->
     </ros2_control>
 </robot>
